Commit message: Get rotors properly placed

File: urdf/dexi.urdf (robot description, URDF)
Before this commit: robot dexi, 12 links, 11 joints
Joints:
- joint base_rotor_1_joint: origin xyz=0.1 -0.1 0 rpy=0 0 0 -> xyz=0.075 -0.095 0 rpy=0 0 0
- joint base_rotor_2_joint: origin xyz=-0.1 0.1 0 rpy=0 0 0 -> xyz=-0.075 0.095 0 rpy=0 0 0
- joint base_rotor_3_joint: origin xyz=0.1 0.1 0 rpy=0 0 0 -> xyz=0.075 0.095 0 rpy=0 0 0
- joint base_rotor_4_joint: origin xyz=-0.1 -0.1 0 rpy=0 0 0 -> xyz=-0.075 -0.095 0 rpy=0 0 0

Commit message: Props WIP

File: urdf/dexi.urdf (robot description, URDF)
Before this commit: robot dexi, 12 links, 11 joints
Links:
- link rotor_1_propeller_link: geometry visual mesh filename=package://dexi_robot_description/meshes/gemfan_ccw.stl scale=0.001 0.001 0.001
- link rotor_3_propeller_link: geometry visual mesh filename=package://dexi_robot_description/meshes/gemfan_cw.stl scale=0.001 0.001 0.001
Joints:
- removed joint rotor_1_propeller_link
- removed joint rotor_2_propeller_link
- removed joint rotor_3_propeller_link
- removed joint rotor_4_propeller_link
- added joint rotor_1_propeller_joint: type fixed, parent rotor_1_link, child rotor_1_propeller_link, origin xyz=0 0 0 rpy=0 0 0
- added joint rotor_2_propeller_joint: type fixed, parent rotor_2_link, child rotor_2_propeller_link, origin xyz=0 0 0.013 rpy=0 0 0.01
- added joint rotor_3_propeller_joint: type fixed, parent rotor_3_link, child rotor_3_propeller_link, origin xyz=0 0 0.013 rpy=0 0 0.01
- added joint rotor_4_propeller_joint: type fixed, parent rotor_4_link, child rotor_4_propeller_link, origin xyz=0 0 0.013 rpy=0 0 0.01

Commit message: Getting propellers oriented

File: urdf/dexi.urdf (robot description, URDF)
Before this commit: robot dexi, 12 links, 11 joints
Links:
- link rotor_2_propeller_link: geometry visual mesh filename=package://dexi_robot_description/meshes/gemfan_ccw.stl scale=0.001 0.001 0.001
- link rotor_4_propeller_link: geometry visual mesh filename=package://dexi_robot_description/meshes/gemfan_cw.stl scale=0.001 0.001 0.001

Commit message: Getting rotors in place

File: urdf/dexi.urdf (robot description, URDF)
Before this commit: robot dexi, 12 links, 11 joints
Links:
- link base_link: geometry visual box size=0 0 0
Joints:
- joint base_rotor_1_joint: origin xyz=0.075 -0.095 0 rpy=0 0 0 -> xyz=0.075 -0.095 0.025 rpy=0 0 0
- joint base_rotor_2_joint: origin xyz=-0.075 0.095 0 rpy=0 0 0 -> xyz=-0.075 0.095 0.025 rpy=0 0 0
- joint base_rotor_3_joint: origin xyz=0.075 0.095 0 rpy=0 0 0 -> xyz=0.075 0.095 0.025 rpy=0 0 0
- joint base_rotor_4_joint: origin xyz=-0.075 -0.095 0 rpy=0 0 0 -> xyz=-0.075 -0.095 0.025 rpy=0 0 0
- joint rotor_1_propeller_joint: origin xyz=0 0 0 rpy=0 0 0 -> xyz=0 0 -0.01 rpy=0 0 0
- joint rotor_2_propeller_joint: origin xyz=0 0 0.013 rpy=0 0 0.01 -> xyz=0 0 -0.01 rpy=0 0 0.01
- joint rotor_3_propeller_joint: origin xyz=0 0 0.013 rpy=0 0 0.01 -> xyz=0 0 -0.01 rpy=0 0 0.01
- joint rotor_4_propeller_joint: origin xyz=0 0 0.013 rpy=0 0 0.01 -> xyz=0 0 -0.01 rpy=0 0 0.01

Commit message: Adding standoffs

File: urdf/dexi.urdf (robot description, URDF)
Before this commit: robot dexi, 12 links, 11 joints
Links:
- removed link rotor_1_link
- added link rotor_1_motor_base_link; visual cylinder length=0.01 radius=0.015
- added link rotor_1_motor_shaft_link; visual cylinder length=0.02 radius=0.01
- added link standoffs_link; visual cylinder length=0.035 radius=0.003; visual cylinder length=0.035 radius=0.003
Joints:
- added joint base_rotor_1_motor_shaft_joint: type continuous, parent rotor_1_motor_base_link, child rotor_1_motor_shaft_link, origin xyz=0 0 -0.015 rpy=0 0 0, axis 0 0 1
- added joint standoffs_joint: type fixed, parent base_link, child standoffs_link, origin xyz=0 0 0 rpy=0 0 0
- joint base_rotor_1_joint: child rotor_1_link -> rotor_1_motor_base_link; origin xyz=0.075 -0.095 0.025 rpy=0 0 0 -> xyz=0.075 -0.095 0.03 rpy=0 0 0; parent base_link -> top_plate_link; type continuous -> fixed
- joint rotor_1_propeller_joint: origin xyz=0 0 -0.01 rpy=0 0 0 -> xyz=0 0 0 rpy=0 0 0; parent rotor_1_link -> rotor_1_motor_shaft_link

Commit message: More standoffs

File: urdf/dexi.urdf (robot description, URDF)
Before this commit: robot dexi, 14 links, 13 joints
Links:
- link standoffs_link: geometry visual cylinder length=0.035 radius=0.003; visual cylinder length=0.035 radius=0.003
